File: Krampus.sch (KiCad schematic (older format))
At the start: 22 parts, among them J1 AVR-ISP-6, Q1 Q_NMOS_GSD, Q2 Q_NMOS_GSD, SW1 SW_SPDT_Flipped, SW2 SW_SPDT, U1 ATtiny4-TS-PROG

Commit message: Added copper pours and keepout areas for tongue and eyes. Everything done except edge cuts and revised mouth (want it to be gold)
Parts:
- C1: footprint Capacitor_SMD:C_0805_2012Metric -> Capacitor_SMD:C_1206_3216Metric_Pad1.33x1.80mm_HandSolder
- Q1, Q2: footprint Package_TO_SOT_SMD:SOT-23 -> Alpenglow:SOT-23-3
- R1, R2, R3, R4, R5, R6, R7, R8: footprint Resistor_SMD:R_0805_2012Metric -> Resistor_SMD:R_1206_3216Metric_Pad1.30x1.75mm_HandSolder
Changed lines of the file:
@@
 F 0 "R3" H 7670 2546 50  0000 L CNN
 F 1 "10k" H 7670 2455 50  0000 L CNN
-F 2 "Resistor_SMD:R_0805_2012Metric" H 7600 2500 50  0001 C CNN
+F 2 "Resistor_SMD:R_1206_3216Metric_Pad1.30x1.75mm_HandSolder" H 7600 2500 50  0001 C CNN
 F 3 "~" H 7600 2500 50  0001 C CNN
 	1    7600 2500
@@
 F 0 "R1" H 8170 1646 50  0000 L CNN
 F 1 "470" H 8170 1555 50  0000 L CNN
-F 2 "Resistor_SMD:R_0805_2012Metric" H 8100 1600 50  0001 C CNN
+F 2 "Resistor_SMD:R_1206_3216Metric_Pad1.30x1.75mm_HandSolder" H 8100 1600 50  0001 C CNN
 F 3 "~" H 8100 1600 50  0001 C CNN
 	1    8100 1600
@@
 F 0 "R2" H 8620 1646 50  0000 L CNN
 F 1 "470" H 8620 1555 50  0000 L CNN
-F 2 "Resistor_SMD:R_0805_2012Metric" H 8550 1600 50  0001 C CNN
+F 2 "Resistor_SMD:R_1206_3216Metric_Pad1.30x1.75mm_HandSolder" H 8550 1600 50  0001 C CNN
 F 3 "~" H 8550 1600 50  0001 C CNN
 	1    8550 1600
@@
 F 0 "Q1" H 8404 2346 50  0000 L CNN
 F 1 "Q_NMOS_GSD" H 8404 2255 50  0000 L CNN
-F 2 "Package_TO_SOT_SMD:SOT-23" H 8400 2400 50  0001 C CNN
+F 2 "Alpenglow:SOT-23-3" H 8400 2400 50  0001 C CNN
 F 3 "~" H 8200 2300 50  0001 C CNN
 	1    8200 2300
@@
 F 0 "Q2" H 8454 5096 50  0000 L CNN
 F 1 "Q_NMOS_GSD" H 8454 5005 50  0000 L CNN
-F 2 "Package_TO_SOT_SMD:SOT-23" H 8450 5150 50  0001 C CNN
+F 2 "Alpenglow:SOT-23-3" H 8450 5150 50  0001 C CNN
 F 3 "~" H 8250 5050 50  0001 C CNN
 	1    8250 5050
@@
 F 0 "R8" H 7720 5346 50  0000 L CNN
 F 1 "10k" H 7720 5255 50  0000 L CNN
-F 2 "Resistor_SMD:R_0805_2012Metric" H 7650 5300 50  0001 C CNN
+F 2 "Resistor_SMD:R_1206_3216Metric_Pad1.30x1.75mm_HandSolder" H 7650 5300 50  0001 C CNN
 F 3 "~" H 7650 5300 50  0001 C CNN
 	1    7650 5300
@@
 F 0 "R4" H 7870 4296 50  0000 L CNN
 F 1 "470" H 7870 4205 50  0000 L CNN
-F 2 "Resistor_SMD:R_0805_2012Metric" H 7800 4250 50  0001 C CNN
+F 2 "Resistor_SMD:R_1206_3216Metric_Pad1.30x1.75mm_HandSolder" H 7800 4250 50  0001 C CNN
 F 3 "~" H 7800 4250 50  0001 C CNN
 	1    7800 4250
@@
 F 0 "R5" H 8220 4296 50  0000 L CNN
 F 1 "470" H 8220 4205 50  0000 L CNN
-F 2 "Resistor_SMD:R_0805_2012Metric" H 8150 4250 50  0001 C CNN
+F 2 "Resistor_SMD:R_1206_3216Metric_Pad1.30x1.75mm_HandSolder" H 8150 4250 50  0001 C CNN
 F 3 "~" H 8150 4250 50  0001 C CNN
 	1    8150 4250
@@
 F 0 "R7" H 8920 4296 50  0000 L CNN
 F 1 "470" H 8920 4205 50  0000 L CNN
-F 2 "Resistor_SMD:R_0805_2012Metric" H 8850 4250 50  0001 C CNN
+F 2 "Resistor_SMD:R_1206_3216Metric_Pad1.30x1.75mm_HandSolder" H 8850 4250 50  0001 C CNN
 F 3 "~" H 8850 4250 50  0001 C CNN
 	1    8850 4250
@@
 F 0 "R6" H 8570 4296 50  0000 L CNN
 F 1 "470" H 8570 4205 50  0000 L CNN
-F 2 "Resistor_SMD:R_0805_2012Metric" H 8500 4250 50  0001 C CNN
+F 2 "Resistor_SMD:R_1206_3216Metric_Pad1.30x1.75mm_HandSolder" H 8500 4250 50  0001 C CNN
 F 3 "~" H 8500 4250 50  0001 C CNN
 	1    8500 4250
@@
 F 0 "C1" H 4781 2096 50  0000 L CNN
 F 1 "0.1" H 4781 2005 50  0000 L CNN
-F 2 "Capacitor_SMD:C_0805_2012Metric" H 4738 1920 50  0001 C CNN
+F 2 "Capacitor_SMD:C_1206_3216Metric_Pad1.33x1.80mm_HandSolder" H 4738 1920 50  0001 C CNN
 F 3 "~" H 4700 2050 50  0001 C CNN
 	1    4700 2050

Commit message: updated sch for final values, added pdfs for schematic and assembly, updated readme for next version notes, added template to schematic, added BOM
Parts:
- BT1: value Battery_Cell -> CR2032
- D1, D2, D3, D4, D5, D6: value LED -> RED
- Q1, Q2: value Q_NMOS_GSD -> N, 2N7002
- R1, R2, R4, R5, R6, R7: value 470 -> 220
- R3, R8: value 10k -> 100k
- SW1: symbol Alpenglow:SW_SPDT_Flipped -> Krampus-rescue:SW_SPDT_Flipped-Alpenglow
Other:
- note added: "MODE SWITCH:\nWICKED FLICKER OR SLOW GLOW"
- note added: "ON/OFF"
- note added: "PROGRAMMING"
Changed lines of the file:
@@
 encoding utf-8
 Sheet 1 1
-Title "Krampus"
+Title "Merry Krampus"
 Date "2021-11-05"
 Rev "A"
-Comp ""
-Comment1 ""
-Comment2 ""
-Comment3 ""
-Comment4 ""
+Comp "company"
+Comment1 "comment1"
+Comment2 "KRP-0100"
+Comment3 "R. WRIGHT"
+Comment4 "comment4"
 $EndDescr
 $Comp
@@
 P 2000 2050
 F 0 "BT1" H 2118 2146 50  0000 L CNN
-F 1 "Battery_Cell" H 2118 2055 50  0000 L CNN
+F 1 "CR2032" H 2118 2055 50  0000 L CNN
 F 2 "Alpenglow:BatteryHolder_CR2032_SMT" V 2000 2110 50  0001 C CNN
 F 3 "~" V 2000 2110 50  0001 C CNN
@@
 U 1 1 61861C6A
 P 3850 2800
-F 0 "U1" H 3875 3481 50  0000 C CNN
-F 1 "ATtiny4-TS-PROG" H 3875 3390 50  0000 C CNN
+F 0 "U1" H 4350 3250 50  0000 C CNN
+F 1 "ATtiny4-TS-PROG" H 4250 2350 50  0000 C CNN
 F 2 "Alpenglow:SOT-23-6_Handsoldering" H 4550 2050 50  0001 C CIN
 F 3 "http://ww1.microchip.com/downloads/en/DeviceDoc/Atmel-8127-AVR-8-bit-Microcontroller-ATtiny4-ATtiny5-ATtiny9-ATtiny10_Datasheet.pdf" H 3850 2700 50  0001 C CNN
@@
 P 7600 2500
 F 0 "R3" H 7670 2546 50  0000 L CNN
-F 1 "10k" H 7670 2455 50  0000 L CNN
+F 1 "100k" H 7670 2455 50  0000 L CNN
 F 2 "Resistor_SMD:R_1206_3216Metric_Pad1.30x1.75mm_HandSolder" H 7600 2500 50  0001 C CNN
 F 3 "~" H 7600 2500 50  0001 C CNN
@@
 P 8100 1600
 F 0 "R1" H 8170 1646 50  0000 L CNN
-F 1 "470" H 8170 1555 50  0000 L CNN
+F 1 "220" H 8170 1555 50  0000 L CNN
 F 2 "Resistor_SMD:R_1206_3216Metric_Pad1.30x1.75mm_HandSolder" H 8100 1600 50  0001 C CNN
 F 3 "~" H 8100 1600 50  0001 C CNN
@@
 P 8550 1600
 F 0 "R2" H 8620 1646 50  0000 L CNN
-F 1 "470" H 8620 1555 50  0000 L CNN
+F 1 "220" H 8620 1555 50  0000 L CNN
 F 2 "Resistor_SMD:R_1206_3216Metric_Pad1.30x1.75mm_HandSolder" H 8550 1600 50  0001 C CNN
 F 3 "~" H 8550 1600 50  0001 C CNN
@@
 P 8200 2300
 F 0 "Q1" H 8404 2346 50  0000 L CNN
-F 1 "Q_NMOS_GSD" H 8404 2255 50  0000 L CNN
+F 1 "N, 2N7002" H 8404 2255 50  0000 L CNN
 F 2 "Alpenglow:SOT-23-3" H 8400 2400 50  0001 C CNN
 F 3 "~" H 8200 2300 50  0001 C CNN
@@
 P 8250 5050
 F 0 "Q2" H 8454 5096 50  0000 L CNN
-F 1 "Q_NMOS_GSD" H 8454 5005 50  0000 L CNN
+F 1 "N, 2N7002" H 8454 5005 50  0000 L CNN
 F 2 "Alpenglow:SOT-23-3" H 8450 5150 50  0001 C CNN
 F 3 "~" H 8250 5050 50  0001 C CNN
@@
 P 8100 1250
 F 0 "D1" V 8146 1180 50  0000 R CNN
-F 1 "LED" V 8055 1180 50  0000 R CNN
+F 1 "RED" V 8055 1180 50  0000 R CNN
 F 2 "Alpenglow:LED_1204_RTA_2P" V 8100 1250 50  0001 C CNN
 F 3 "~" V 8100 1250 50  0001 C CNN
@@
 P 8550 1250
 F 0 "D2" V 8596 1180 50  0000 R CNN
-F 1 "LED" V 8505 1180 50  0000 R CNN
+F 1 "RED" V 8505 1180 50  0000 R CNN
 F 2 "Alpenglow:LED_1204_RTA_2P" V 8550 1250 50  0001 C CNN
 F 3 "~" V 8550 1250 50  0001 C CNN
@@
 P 7650 5300
 F 0 "R8" H 7720 5346 50  0000 L CNN
-F 1 "10k" H 7720 5255 50  0000 L CNN
+F 1 "100k" H 7720 5255 50  0000 L CNN
 F 2 "Resistor_SMD:R_1206_3216Metric_Pad1.30x1.75mm_HandSolder" H 7650 5300 50  0001 C CNN
 F 3 "~" H 7650 5300 50  0001 C CNN
@@
 P 7800 4250
 F 0 "R4" H 7870 4296 50  0000 L CNN
-F 1 "470" H 7870 4205 50  0000 L CNN
+F 1 "220" H 7870 4205 50  0000 L CNN
 F 2 "Resistor_SMD:R_1206_3216Metric_Pad1.30x1.75mm_HandSolder" H 7800 4250 50  0001 C CNN
 F 3 "~" H 7800 4250 50  0001 C CNN
@@
 P 8150 4250
 F 0 "R5" H 8220 4296 50  0000 L CNN
-F 1 "470" H 8220 4205 50  0000 L CNN
+F 1 "220" H 8220 4205 50  0000 L CNN
 F 2 "Resistor_SMD:R_1206_3216Metric_Pad1.30x1.75mm_HandSolder" H 8150 4250 50  0001 C CNN
 F 3 "~" H 8150 4250 50  0001 C CNN
@@
 P 8850 4250
 F 0 "R7" H 8920 4296 50  0000 L CNN
-F 1 "470" H 8920 4205 50  0000 L CNN
+F 1 "220" H 8920 4205 50  0000 L CNN
 F 2 "Resistor_SMD:R_1206_3216Metric_Pad1.30x1.75mm_HandSolder" H 8850 4250 50  0001 C CNN
 F 3 "~" H 8850 4250 50  0001 C CNN
@@
 P 8500 4250
 F 0 "R6" H 8570 4296 50  0000 L CNN
-F 1 "470" H 8570 4205 50  0000 L CNN
+F 1 "220" H 8570 4205 50  0000 L CNN
 F 2 "Resistor_SMD:R_1206_3216Metric_Pad1.30x1.75mm_HandSolder" H 8500 4250 50  0001 C CNN
 F 3 "~" H 8500 4250 50  0001 C CNN
@@
 P 7800 3900
 F 0 "D3" V 7846 3830 50  0000 R CNN
-F 1 "LED" V 7755 3830 50  0000 R CNN
+F 1 "RED" V 7755 3830 50  0000 R CNN
 F 2 "Alpenglow:LED_1204_RTA_2P" V 7800 3900 50  0001 C CNN
 F 3 "~" V 7800 3900 50  0001 C CNN
@@
 P 8150 3900
 F 0 "D4" V 8196 3830 50  0000 R CNN
-F 1 "LED" V 8105 3830 50  0000 R CNN
+F 1 "RED" V 8105 3830 50  0000 R CNN
 F 2 "Alpenglow:LED_1204_RTA_2P" V 8150 3900 50  0001 C CNN
 F 3 "~" V 8150 3900 50  0001 C CNN
@@
 P 8500 3900
 F 0 "D5" V 8546 3830 50  0000 R CNN
-F 1 "LED" V 8455 3830 50  0000 R CNN
+F 1 "RED" V 8455 3830 50  0000 R CNN
 F 2 "Alpenglow:LED_1204_RTA_2P" V 8500 3900 50  0001 C CNN
 F 3 "~" V 8500 3900 50  0001 C CNN
@@
 P 8850 3900
 F 0 "D6" V 8896 3830 50  0000 R CNN
-F 1 "LED" V 8805 3830 50  0000 R CNN
+F 1 "RED" V 8805 3830 50  0000 R CNN
 F 2 "Alpenglow:LED_1204_RTA_2P" V 8850 3900 50  0001 C CNN
 F 3 "~" V 8850 3900 50  0001 C CNN
@@
 P 7950 6100
 F 0 "SW2" H 7950 6385 50  0000 C CNN
-F 1 "SW_SPDT" H 7950 6294 50  0000 C CNN
+F 1 "SW_SPDT" H 7950 6294 50  0001 C CNN
 F 2 "Button_Switch_SMD:SW_SPDT_PCM12" H 7950 6100 50  0001 C CNN
 F 3 "~" H 7950 6100 50  0001 C CNN
@@
 TONGUE
 $Comp
-L Alpenglow:SW_SPDT_Flipped SW1
+L Krampus-rescue:SW_SPDT_Flipped-Alpenglow SW1
 U 1 1 61860744
 P 3200 1700
 F 0 "SW1" H 3200 1985 50  0000 C CNN
-F 1 "SW_SPDT_Flipped" H 3200 1894 50  0000 C CNN
+F 1 "SW_SPDT_Flipped" H 3200 1894 50  0001 C CNN
 F 2 "Button_Switch_SMD:SW_SPDT_PCM12" H 3200 1700 50  0001 C CNN
 F 3 "~" H 3200 1700 50  0001 C CNN
@@
 Wire Wire Line
 	3850 1600 3850 1350
+Text Notes 8550 6100 0    50   ~ 0
+MODE SWITCH:\nWICKED FLICKER OR SLOW GLOW
+Text Notes 2650 6150 0    50   ~ 0
+PROGRAMMING
+Text Notes 3050 2050 0    50   ~ 0
+ON/OFF
 $EndSCHEMATC
