File: Krampus.kicad_pcb (KiCad board)
At the start: 2 copper layers, 67.3 x 117.5 mm, 31 parts, among them J1 AVR-ISP-6, Q1 Q_NMOS_GSD, Q2 Q_NMOS_GSD, SW1 SW_SPDT_Flipped, SW2 SW_SPDT, U1 ATtiny4-TS-PROG

Commit message: Updated board name with font, updated @alpenglowind to oswald font
Parts:
- added G***: LOGO, Krampus:KRP board name font 20x2.9mm, B.Cu at (79.8, 136.1)
- added G***: LOGO, Alpenglow:@AlpenglowIndOswald20mm, B.Cu at (41.4, 50.3)
Other:
- net class Default removed
- board text removed: "@AlpenglowInd"
- board text removed: "Merry Krampus!"

Commit message: Changed 10k resistor value to 100k
Parts:
- R3, R8: value 10k -> 100k
Changed lines of the file:
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@@
       (effects (font (size 1.524 1.524) (thickness 0.1778)) (justify mirror))
     )
-    (fp_text value "10k" (at 0 -1.82 90) (layer "B.SilkS")
-      (effects (font (size 1.524 1.524) (thickness 0.1778)) (justify mirror))
+    (fp_text value "100k" (at 0 -2.159 90) (layer "B.SilkS")
+      (effects (font (size 1.016 1.016) (thickness 0.1524)) (justify mirror))
     )
     (fp_text user "${REFERENCE}" (at 0 0 90) (layer "B.Fab")
@@
       (effects (font (size 1.524 1.524) (thickness 0.1778)) (justify mirror))
     )
-    (fp_text value "10k" (at 0 -1.82 90) (layer "B.SilkS")
-      (effects (font (size 1.524 1.524) (thickness 0.1778)) (justify mirror))
+    (fp_text value "100k" (at 0 -2.159 90) (layer "B.SilkS")
+      (effects (font (size 1.016 1.016) (thickness 0.1524)) (justify mirror))
     )
     (fp_text user "${REFERENCE}" (at 0 0 90) (layer "B.Fab")
@@
   (gr_line (start 94.243639 86.052636) (end 94.348972 85.822616) (layer "Edge.Cuts") (width 0.00208))
   (gr_arc (start 41.488188 66.578075) (mid 42.06398 67.604067) (end 42.542484 68.678884) (layer "Edge.Cuts") (width 0.00208))
-  (gr_arc (start 102.936913 43.832308) (mid 103.233964 44.885891) (end 103.452795 45.958452) (layer "Edge.Cuts") (width 0.00208))
+  (gr_arc (start 102.936913 43.832308) (mid 103.233964 44.88589) (end 103.452795 45.958452) (layer "Edge.Cuts") (width 0.00208))
   (gr_line (start 39.729287 44.377452) (end 39.547276 44.873998) (layer "Edge.Cuts") (width 0.00208))
   (gr_arc (start 78.015106 146.503424) (mid 77.863733 146.917553) (end 77.672224 147.31472) (layer "Edge.Cuts") (width 0.00208))
@@
   (gr_line (start 93.080484 53.01365) (end 92.47245 54.052707) (layer "Edge.Cuts") (width 0.00208))
   (gr_arc (start 103.836077 56.441306) (mid 103.698966 56.678092) (end 103.540831 56.901386) (layer "Edge.Cuts") (width 0.00208))
-  (gr_arc (start 94.235098 86.31667) (mid 94.221789 86.251097) (end 94.217326 86.184335) (layer "Edge.Cuts") (width 0.00208))
+  (gr_arc (start 94.235098 86.31667) (mid 94.221789 86.251096) (end 94.217326 86.184335) (layer "Edge.Cuts") (width 0.00208))
   (gr_arc (start 47.232264 88.301975) (mid 47.252475 87.962715) (end 47.29442 87.625452) (layer "Edge.Cuts") (width 0.00208))
   (gr_arc (start 90.701461 114.109765) (mid 90.753152 114.01118) (end 90.814947 113.918592) (layer "Edge.Cuts") (width 0.00208))
@@
   (gr_arc (start 95.325055 84.043015) (mid 95.193795 84.360511) (end 95.042108 84.66877) (layer "Edge.Cuts") (width 0.00208))
   (gr_arc (start 49.567314 97.965332) (mid 49.59859 97.615445) (end 49.646197 97.267404) (layer "Edge.Cuts") (width 0.00208))
-  (gr_arc (start 50.862697 31.540449) (mid 51.505962 31.32075) (end 52.169191 31.171799) (layer "Edge.Cuts") (width 0.00208))
+  (gr_arc (start 50.862697 31.540449) (mid 51.505963 31.32075) (end 52.169191 31.171799) (layer "Edge.Cuts") (width 0.00208))
   (gr_line (start 59.842271 134.723001) (end 60.25643 135.276848) (layer "Edge.Cuts") (width 0.00208))
   (gr_line (start 56.408459 129.007989) (end 56.60659 129.257886) (layer "Edge.Cuts") (width 0.00208))
@@
   (gr_line (start 52.813966 118.463557) (end 53.162953 119.231874) (layer "Edge.Cuts") (width 0.00208))
   (gr_arc (start 49.741786 93.449217) (mid 49.944736 93.602466) (end 50.127119 93.779696) (layer "Edge.Cuts") (width 0.00208))
-  (gr_arc (start 55.51613 37.56233) (mid 55.71018 37.193387) (end 55.922356 36.834563) (layer "Edge.Cuts") (width 0.00208))
+  (gr_arc (start 55.51613 37.56233) (mid 55.71018 37.193388) (end 55.922356 36.834563) (layer "Edge.Cuts") (width 0.00208))
   (gr_line (start 95.943235 81.515281) (end 96.137651 81.36557) (layer "Edge.Cuts") (width 0.00208))
   (gr_arc (start 77.24676 147.900101) (mid 76.986598 148.13873) (end 76.695572 148.33856) (layer "Edge.Cuts") (width 0.00208))
@@
   (gr_arc (start 78.348608 64.784664) (mid 77.965727 64.950242) (end 77.575812 65.098499) (layer "Edge.Cuts") (width 0.00208))
   (gr_line (start 104.453801 54.976444) (end 104.745737 54.050549) (layer "Edge.Cuts") (width 0.00208))
-  (gr_arc (start 49.663776 32.181395) (mid 50.245958 31.8286) (end 50.862697 31.540448) (layer "Edge.Cuts") (width 0.00208))
+  (gr_arc (start 49.663776 32.181395) (mid 50.245957 31.8286) (end 50.862697 31.540448) (layer "Edge.Cuts") (width 0.00208))
   (gr_line (start 39.172187 63.43656) (end 39.389989 63.754683) (layer "Edge.Cuts") (width 0.00208))
   (gr_line (start 55.442922 60.907654) (end 54.063166 59.628526) (layer "Edge.Cuts") (width 0.00208))
@@
   (gr_arc (start 51.381363 113.364878) (mid 51.474356 113.577026) (end 51.532715 113.801188) (layer "Edge.Cuts") (width 0.00208))
   (gr_arc (start 92.200478 96.412855) (mid 92.125106 96.051684) (end 92.065939 95.687508) (layer "Edge.Cuts") (width 0.00208))
-  (gr_arc (start 47.38391 89.663422) (mid 47.310892 89.315268) (end 47.260102 88.963185) (layer "Edge.Cuts") (width 0.00208))
+  (gr_arc (start 47.38391 89.663422) (mid 47.310892 89.315269) (end 47.260102 88.963185) (layer "Edge.Cuts") (width 0.00208))
   (gr_line (start 49.200401 81.905468) (end 49.28377 82.184483) (layer "Edge.Cuts") (width 0.00208))
   (gr_line (start 50.838989 43.625037) (end 51.319758 43.378463) (layer "Edge.Cuts") (width 0.00208))

Commit message: Added On OFF labels and pin1 mark on back silkscreen
Other:
- board text added: "OFF"
- board text added: "ON"
Changed lines of the file:
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@@
       ) (layer "B.SilkS") (width 0) (fill solid))
   )
+  (gr_circle (center 77.724 110.236) (end 78.105 110.236) (layer "B.SilkS") (width 0.12) (fill solid))
   (gr_line (start 48.657034 48.240102) (end 48.701561 47.496791) (layer "Edge.Cuts") (width 0.00208))
   (gr_line (start 94.49391 85.558041) (end 94.665485 85.289831) (layer "Edge.Cuts") (width 0.00208))
@@
   (gr_line (start 95.741432 82.227026) (end 95.799067 81.917164) (layer "Edge.Cuts") (width 0.00208))
   (gr_arc (start 48.545074 80.623214) (mid 48.691118 80.721238) (end 48.817041 80.844044) (layer "Edge.Cuts") (width 0.00208))
+  (gr_text "OFF" (at 44.069 64.897 10) (layer "B.SilkS")
+    (effects (font (size 1.143 1.143) (thickness 0.1524)) (justify mirror))
+  )
+  (gr_text "ON" (at 46.101 76.454 10) (layer "B.SilkS")
+    (effects (font (size 1.143 1.143) (thickness 0.1524)) (justify mirror))
+  )
   (segment (start 61.595 108.966) (end 61.722 108.839) (width 0.254) (layer "F.Cu") (net 1))
   (segment (start 83.566 120.523) (end 79.883 120.523) (width 0.254) (layer "F.Cu") (net 1))
